File: examples/rf_diffvia.kicad_pcb (KiCad board)
At the start: 4 copper layers, 24 x 8 mm, 4 parts

Commit message: Line model: differential pairs couple, qucsator's missing terms are zero; rf_diffvia with two nets
- Coupled sections: the ends of the overlaps are merged within 1 um before cutting, and the pieces are keyed
  by their cut: rounding to 0.1 um had put two legs starting at 0.57424999 and 0.57425 mm into different
  pieces, so a pair laid out by coordinates never coupled. The filters' coupled sections are unchanged.
- qucsator leaves out the S-parameters between separate circuits (two legs not coupled): read as 0, not a
  KeyError.
- make_rf_examples.diffvia: the legs on nets D_P / D_N, as a real pair.

Co-Authored-By: Claude Opus 5.5 <noreply@anthropic.com>
Claude-Session: https://claude.ai/code/session_01TtsBLmmPmy9tKEvcwxPT5D
Routing:
- net RF: track 48.3 -> 0.00 mm, vias 2 -> 0
- net D_P: track 0.00 -> 24.2 mm, vias 0 -> 1
- net D_N: track 0.00 -> 24.2 mm, vias 0 -> 1
Changed lines of the file:
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@@
     (copper_finish "None") (dielectric_constraints no))
     (pad_to_mask_clearance 0))
-  (net 0 "") (net 1 "GND") (net 2 "RF")
+  (net 0 "") (net 1 "GND") (net 2 "D_P") (net 3 "D_N")
   (segment (start 0.0000 3.7515) (end 10.5000 3.7515) (width 0.297) (layer "F.Cu") (net 2))
   (segment (start 10.5000 3.7515) (end 11.0000 3.5000) (width 0.297) (layer "F.Cu") (net 2))
@@
   (via (at 11.1000 2.6000) (size 0.5) (drill 0.25) (layers "F.Cu" "B.Cu") (net 1))
   (via (at 12.9000 2.6000) (size 0.5) (drill 0.25) (layers "F.Cu" "B.Cu") (net 1))
-  (segment (start 0.0000 4.2485) (end 10.5000 4.2485) (width 0.297) (layer "F.Cu") (net 2))
-  (segment (start 10.5000 4.2485) (end 11.0000 4.5000) (width 0.297) (layer "F.Cu") (net 2))
-  (segment (start 11.0000 4.5000) (end 12.0000 4.5000) (width 0.297) (layer "F.Cu") (net 2))
-  (segment (start 12.0000 4.5000) (end 13.0000 4.5000) (width 0.157) (layer "In2.Cu") (net 2))
-  (segment (start 13.0000 4.5000) (end 13.5000 4.1785) (width 0.157) (layer "In2.Cu") (net 2))
-  (segment (start 13.5000 4.1785) (end 24.0000 4.1785) (width 0.157) (layer "In2.Cu") (net 2))
-  (via blind (at 12.0000 4.5000) (size 0.5) (drill 0.25) (layers "F.Cu" "In2.Cu") (net 2))
+  (segment (start 0.0000 4.2485) (end 10.5000 4.2485) (width 0.297) (layer "F.Cu") (net 3))
+  (segment (start 10.5000 4.2485) (end 11.0000 4.5000) (width 0.297) (layer "F.Cu") (net 3))
+  (segment (start 11.0000 4.5000) (end 12.0000 4.5000) (width 0.297) (layer "F.Cu") (net 3))
+  (segment (start 12.0000 4.5000) (end 13.0000 4.5000) (width 0.157) (layer "In2.Cu") (net 3))
+  (segment (start 13.0000 4.5000) (end 13.5000 4.1785) (width 0.157) (layer "In2.Cu") (net 3))
+  (segment (start 13.5000 4.1785) (end 24.0000 4.1785) (width 0.157) (layer "In2.Cu") (net 3))
+  (via blind (at 12.0000 4.5000) (size 0.5) (drill 0.25) (layers "F.Cu" "In2.Cu") (net 3))
   (via (at 11.1000 5.4000) (size 0.5) (drill 0.25) (layers "F.Cu" "B.Cu") (net 1))
   (via (at 12.9000 5.4000) (size 0.5) (drill 0.25) (layers "F.Cu" "B.Cu") (net 1))
